Commit message: 调整灭火器结构

File: TienKung-Lab/legged_lab/assets/h1_description/urdf/h1_payload_horizontal.urdf (robot description, URDF)
Before this commit: robot h1_payload_horizontal, 32 links, 31 joints
Links:
- link h1_extinguisher_payload: geometry collision box size=0.062 0.405 0.062; visual box size=0.062 0.405 0.062
Joints:
- joint payload_mount_x_joint: origin xyz=-0.18 0 0.10 rpy=0 0 0 -> xyz=-0.18 0 0.05 rpy=0 0 0
